File: hardware/gw.kicad_pcb (KiCad board)
At the start: 4 copper layers, 47 x 32.9 mm, 21 parts, among them J1 USB_OTG, J2 Conn_01x04, U1 ESP-12F, U2 Ai-Thinker-Ra-02, U3 AMS1117-3.3

Commit message: Latest fixes
Connections:
- J2 pad 3: /RXD_D0 -> /RXD
- R5 pad 1: /DIO1 -> /DIO0
- U1 pad 11: /DIO1 -> /DIO0
- U1 pad 15: /RXD_D0 -> /RXD
- U2 pad 5: /RXD_D0 -> /DIO0
- U2 pad 6: /DIO1 -> unconnected-(U2-Pad6)
Routing:
- net /RXD_D0: track 45.6 -> 0.00 mm, vias 2 -> 0
- net /DIO0: track 0.00 -> 32.7 mm, vias 0 -> 2
- net /DIO1: track 30.6 -> 0.00 mm, vias 2 -> 0
- net /RXD: track 0.00 -> 7.59 mm
- net /DIO2: track 29.0 -> 28.5 mm
Changed lines of the file:
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@@
   (net 23 "/WF_LED")
   (net 24 "/DIO2")
-  (net 25 "/DIO1")
+  (net 25 "/RXD")
   (net 26 "/SS")
-  (net 27 "/RXD_D0")
+  (net 27 "/DIO0")
+  (net 28 "unconnected-(U2-Pad6)")
   (footprint "LED_SMD:LED_1206_3216Metric" (layer "F.Cu")
     (at 92.35 72.7 180)
@@
       (net 1 "/RESET") (pinfunction "~{RESET}") (pintype "input"))
     (pad "5" smd rect (at -8 1 90) (size 2 1.5) (layers "F.Cu" "F.Paste" "F.Mask")
-      (net 27 "/RXD_D0") (pinfunction "DIO0") (pintype "bidirectional"))
+      (net 27 "/DIO0") (pinfunction "DIO0") (pintype "bidirectional"))
     (pad "6" smd rect (at -8 3 90) (size 2 1.5) (layers "F.Cu" "F.Paste" "F.Mask")
-      (net 25 "/DIO1") (pinfunction "DIO1") (pintype "bidirectional"))
+      (net 28 "unconnected-(U2-Pad6)") (pinfunction "DIO1") (pintype "bidirectional+no_connect"))
     (pad "7" smd rect (at -8 5 90) (size 2 1.5) (layers "F.Cu" "F.Paste" "F.Mask")
       (net 24 "/DIO2") (pinfunction "DIO2") (pintype "bidirectional"))
@@
       (net 1 "/RESET") (pinfunction "GPIO15") (pintype "bidirectional"))
     (pad "11" smd rect (at 7.6 5.1) (size 2.5 1) (layers "F.Cu" "F.Paste" "F.Mask")
-      (net 25 "/DIO1") (pinfunction "GPIO2") (pintype "bidirectional"))
+      (net 27 "/DIO0") (pinfunction "GPIO2") (pintype "bidirectional"))
     (pad "12" smd rect (at 7.6 3.1) (size 2.5 1) (layers "F.Cu" "F.Paste" "F.Mask")
       (net 23 "/WF_LED") (pinfunction "GPIO0") (pintype "bidirectional"))
@@
       (net 26 "/SS") (pinfunction "GPIO5") (pintype "bidirectional"))
     (pad "15" smd rect (at 7.6 -2.9) (size 2.5 1) (layers "F.Cu" "F.Paste" "F.Mask")
-      (net 27 "/RXD_D0") (pinfunction "GPIO3/RXD") (pintype "bidirectional"))
+      (net 25 "/RXD") (pinfunction "GPIO3/RXD") (pintype "bidirectional"))
     (pad "16" smd rect (at 7.6 -4.9) (size 2.5 1) (layers "F.Cu" "F.Paste" "F.Mask")
       (net 20 "/TXD") (pinfunction "GPIO1/TXD") (pintype "bidirectional"))
@@
     (fp_line (start 1.6 0.8) (end -1.6 0.8) (layer "F.Fab") (width 0.1))
     (pad "1" smd roundrect (at -1.4625 0 90) (size 1.125 1.75) (layers "F.Cu" "F.Paste" "F.Mask") (roundrect_rratio 0.2222222222)
-      (net 25 "/DIO1") (pintype "passive"))
+      (net 27 "/DIO0") (pintype "passive"))
     (pad "2" smd roundrect (at 1.4625 0 90) (size 1.125 1.75) (layers "F.Cu" "F.Paste" "F.Mask") (roundrect_rratio 0.2222222222)
       (net 7 "+3V3") (pintype "passive"))
@@
       (net 6 "GND") (pinfunction "Pin_2") (pintype "passive"))
     (pad "3" thru_hole oval (at 0 5.08 180) (size 1.7 1.7) (drill 1) (layers *.Cu *.Mask)
-      (net 27 "/RXD_D0") (pinfunction "Pin_3") (pintype "passive"))
+      (net 25 "/RXD") (pinfunction "Pin_3") (pintype "passive"))
     (pad "4" thru_hole oval (at 0 7.62 180) (size 1.7 1.7) (drill 1) (layers *.Cu *.Mask)
       (net 20 "/TXD") (pinfunction "Pin_4") (pintype "passive"))
@@
   (segment (start 93.8 67.3) (end 93.8 67.5) (width 0.25) (layer "B.Cu") (net 23))
   (segment (start 89.652606 53.947394) (end 86.55 57.05) (width 0.25) (layer "B.Cu") (net 23))
-  (segment (start 110.61 51.95) (end 109.728 52.832) (width 0.25) (layer "F.Cu") (net 24))
+  (segment (start 109.6772 56.2102) (end 108.7628 57.1246) (width 0.25) (layer "F.Cu") (net 24))
   (segment (start 94.2964 59.6536) (end 94.3 59.65) (width 0.25) (layer "F.Cu") (net 24))
   (segment (start 94.2964 61.2694) (end 94.2964 59.6536) (width 0.25) (layer "F.Cu") (net 24))
-  (segment (start 109.728 57.15) (end 109.728 52.832) (width 0.25) (layer "F.Cu") (net 24))
-  (segment (start 108.966 57.912) (end 109.728 57.15) (width 0.25) (layer "F.Cu") (net 24))
   (segment (start 116 51.95) (end 110.61 51.95) (width 0.25) (layer "F.Cu") (net 24))
+  (segment (start 108.7628 57.1246) (end 107.823 57.1246) (width 0.25) (layer "F.Cu") (net 24))
+  (segment (start 110.61 51.95) (end 109.6772 52.8828) (width 0.25) (layer "F.Cu") (net 24))
+  (segment (start 109.6772 52.8828) (end 109.6772 56.2102) (width 0.25) (layer "F.Cu") (net 24))
   (via (at 94.3 59.65) (size 0.45) (drill 0.2) (layers "F.Cu" "B.Cu") (net 24))
-  (via (at 108.966 57.912) (size 0.45) (drill 0.2) (layers "F.Cu" "B.Cu") (net 24))
-  (segment (start 108.966 57.912) (end 96.038 57.912) (width 0.25) (layer "B.Cu") (net 24))
-  (segment (start 96.038 57.912) (end 94.3 59.65) (width 0.25) (layer "B.Cu") (net 24))
-  (segment (start 116 55.95) (end 114.125 55.95) (width 0.25) (layer "F.Cu") (net 25))
-  (segment (start 116.0214 55.9694) (end 118.681 55.9694) (width 0.25) (layer "F.Cu") (net 25))
-  (segment (start 93.1164 59.0296) (end 92.2964 59.8496) (width 0.25) (layer "F.Cu") (net 25))
-  (segment (start 118.681 55.9694) (end 119.507 55.1434) (width 0.25) (layer "F.Cu") (net 25))
-  (segment (start 96.8756 59.0296) (end 93.1164 59.0296) (width 0.25) (layer "F.Cu") (net 25))
-  (segment (start 92.2964 61.2694) (end 92.2964 59.8496) (width 0.25) (layer "F.Cu") (net 25))
-  (via (at 96.8756 59.0296) (size 0.45) (drill 0.2) (layers "F.Cu" "B.Cu") (net 25))
-  (via (at 114.125 55.95) (size 0.45) (drill 0.2) (layers "F.Cu" "B.Cu") (net 25))
-  (segment (start 112.96 55.95) (end 109.8804 59.0296) (width 0.25) (layer "B.Cu") (net 25))
-  (segment (start 109.8804 59.0296) (end 96.8756 59.0296) (width 0.25) (layer "B.Cu") (net 25))
-  (segment (start 114.125 55.95) (end 112.96 55.95) (width 0.25) (layer "B.Cu") (net 25))
+  (via (at 107.823 57.1246) (size 0.45) (drill 0.2) (layers "F.Cu" "B.Cu") (net 24))
+  (segment (start 96.8254 57.1246) (end 107.823 57.1246) (width 0.25) (layer "B.Cu") (net 24))
+  (segment (start 94.3 59.65) (end 96.8254 57.1246) (width 0.25) (layer "B.Cu") (net 24))
+  (segment (start 116.0214 47.9694) (end 122.0966 47.9694) (width 0.25) (layer "F.Cu") (net 25))
+  (segment (start 122.0966 47.9694) (end 123.1646 49.0374) (width 0.25) (layer "F.Cu") (net 25))
   (segment (start 113.0046 48.8188) (end 111.5568 48.8188) (width 0.25) (layer "F.Cu") (net 26))
   (segment (start 84.2964 47.274284) (end 84.306084 47.283968) (width 0.25) (layer "F.Cu") (net 26))
@@
   (segment (start 84.306084 48.238084) (end 84.306084 47.283968) (width 0.25) (layer "B.Cu") (net 26))
   (segment (start 84.8868 48.8188) (end 84.306084 48.238084) (width 0.25) (layer "B.Cu") (net 26))
-  (segment (start 107.8992 56.6674) (end 107.823 56.6674) (width 0.25) (layer "F.Cu") (net 27))
-  (segment (start 108.4326 56.134) (end 108.4326 48.5394) (width 0.25) (layer "F.Cu") (net 27))
-  (segment (start 114.046 47.3456) (end 109.6264 47.3456) (width 0.25) (layer "F.Cu") (net 27))
+  (segment (start 116 55.95) (end 114.125 55.95) (width 0.25) (layer "F.Cu") (net 27))
+  (segment (start 90.935798 59.0296) (end 90.294802 59.670596) (width 0.25) (layer "F.Cu") (net 27))
+  (segment (start 116.0214 55.9694) (end 118.681 55.9694) (width 0.25) (layer "F.Cu") (net 27))
+  (segment (start 96.8756 59.0296) (end 90.935798 59.0296) (width 0.25) (layer "F.Cu") (net 27))
   (segment (start 90.2964 59.672194) (end 90.294802 59.670596) (width 0.25) (layer "F.Cu") (net 27))
-  (segment (start 109.6264 47.3456) (end 108.4326 48.5394) (width 0.25) (layer "F.Cu") (net 27))
-  (segment (start 114.6504 47.95) (end 114.046 47.3456) (width 0.25) (layer "F.Cu") (net 27))
-  (segment (start 116.0214 47.9694) (end 122.0966 47.9694) (width 0.25) (layer "F.Cu") (net 27))
+  (segment (start 118.681 55.9694) (end 119.507 55.1434) (width 0.25) (layer "F.Cu") (net 27))
   (segment (start 90.2964 61.2694) (end 90.2964 59.672194) (width 0.25) (layer "F.Cu") (net 27))
-  (segment (start 122.0966 47.9694) (end 123.1646 49.0374) (width 0.25) (layer "F.Cu") (net 27))
-  (segment (start 108.4326 56.134) (end 107.8992 56.6674) (width 0.25) (layer "F.Cu") (net 27))
-  (segment (start 116 47.95) (end 114.6504 47.95) (width 0.25) (layer "F.Cu") (net 27))
-  (via (at 107.823 56.6674) (size 0.45) (drill 0.2) (layers "F.Cu" "B.Cu") (net 27))
-  (via (at 90.294802 59.670596) (size 0.45) (drill 0.2) (layers "F.Cu" "B.Cu") (net 27))
-  (segment (start 107.823 56.6674) (end 91.7448 56.6674) (width 0.25) (layer "B.Cu") (net 27))
-  (segment (start 90.294802 58.117398) (end 90.294802 59.670596) (width 0.25) (layer "B.Cu") (net 27))
-  (segment (start 91.7448 56.6674) (end 90.294802 58.117398) (width 0.25) (layer "B.Cu") (net 27))
+  (via (at 96.8756 59.0296) (size 0.45) (drill 0.2) (layers "F.Cu" "B.Cu") (net 27))
+  (via (at 114.125 55.95) (size 0.45) (drill 0.2) (layers "F.Cu" "B.Cu") (net 27))
+  (segment (start 112.96 55.95) (end 109.8804 59.0296) (width 0.25) (layer "B.Cu") (net 27))
+  (segment (start 109.8804 59.0296) (end 96.8756 59.0296) (width 0.25) (layer "B.Cu") (net 27))
+  (segment (start 114.125 55.95) (end 112.96 55.95) (width 0.25) (layer "B.Cu") (net 27))
   (zone (net 7) (net_name "+3V3") (layer "F.Cu") (hatch edge 0.508)
     (connect_pads yes (clearance 0.508))

Commit message: Fixup pins
Connections:
- R5 pad 1: /DIO0 -> /SS
- U1 pad 11: /DIO0 -> /SS
- U1 pad 14: /SS -> /DIO0
Routing:
- net /WF_LED: track 59.5 -> 43.8 mm
- net Net-(R1-Pad2): track 33.6 -> 26.6 mm, vias 0 -> 2
- net /RF_LED: track 20.7 -> 27.2 mm
- net /SS: track 35.4 -> 41.1 mm
- net /RESET: track 36.6 -> 33.4 mm
- net /DIO0: track 32.7 -> 33.3 mm
- net Net-(R3-Pad2): track 24.2 -> 23.6 mm
- net /DIO2: track 28.5 -> 27.8 mm

Commit message: Latest prefab
Other:
- board text added: "BT GND RXD TXD"
Changed lines of the file:
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@@
     (effects (font (size 1 1) (thickness 0.2)))
+  )
+  (gr_text "BT GND RXD TXD" (at 125.0696 45.1866 90) (layer "F.SilkS")
+    (effects (font (size 0.75 0.75) (thickness 0.15)) (justify right))
   )
   (gr_text "S" (at 86.106 70.612) (layer "F.SilkS")

Commit message: Name changes
Parts:
- D1: value RF -> WIFI
- D2: value WIFI -> RF
Connections:
- R2 pad 2: /RF_LED -> /WF_LED
- R4 pad 1: /WF_LED -> /RF_LED
- R8 pad 2: /WF_LED -> /RF_LED
- U1 pad 12: /WF_LED -> /RF_LED
- U1 pad 4: /RF_LED -> /WF_LED
Routing:
- net /WF_LED: track 43.8 -> 27.2 mm
- net /RF_LED: track 27.2 -> 43.8 mm
Other:
- board text added: "RADIO ST"
- board text added: "WIFI ST"
- board text removed: "NET STAT"
- board text removed: "RF STAT"

Commit message: Fix rev
Other:
- board text added: "20 22"
- board text added: "rev: 04a by:"
- board text removed: "rev: m4a by:"
Changed lines of the file:
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@@
     (effects (font (size 0.75 0.75) (thickness 0.15)) (justify right))
   )
-  (gr_text "S" (at 86.106 70.612) (layer "F.SilkS")
+  (gr_text "S" (at 86.175 70.925) (layer "F.SilkS")
     (effects (font (size 2 2) (thickness 0.2)))
   )
@@
     (effects (font (size 0.75 0.75) (thickness 0.15)) (justify right))
   )
-  (gr_text "rev: m4a\nby:" (at 80.264 68.072) (layer "F.SilkS")
+  (gr_text "rev: 04a\nby:" (at 80.264 68.072) (layer "F.SilkS")
     (effects (font (size 1 1) (thickness 0.2)) (justify left))
   )
-  (gr_text "K" (at 84.328 70.104) (layer "F.SilkS")
+  (gr_text "K" (at 84.875 69.975) (layer "F.SilkS")
     (effects (font (size 3 3) (thickness 0.2)))
   )
@@
     (effects (font (size 0.75 0.75) (thickness 0.15)) (justify right))
   )
+  (gr_text "20\n22" (at 81.375 71.675) (layer "F.SilkS")
+    (effects (font (size 1 1) (thickness 0.2)))
+  )
   (dimension (type aligned) (layer "B.Cu")
